Commit message: add imu_link and update urdf

File: pui_description/urdf/pui_bot.urdf (robot description, URDF)
Before this commit: robot pui_bot, 7 links, 6 joints
Links:
- link imu_link: geometry visual mesh filename=package://xsens_mti_driver/urdf/MTi_1.stl scale=0.001 0.001 0.001

Commit message: add velodyne and xsens stl

File: pui_description/urdf/pui_bot.urdf (robot description, URDF)
Before this commit: robot pui_bot, 7 links, 6 joints
Links:
- link base_scan: geometry collision cylinder length=0.0315 radius=0.055; visual mesh filename=package://pui_description/meshes/sensors/vlp.stl scale=0.001 0.001 0.001
- link imu_link: geometry visual mesh filename=package://pui_description/meshes/sensors/MTi_1.stl scale=0.001 0.001 0.001
Joints:
- joint imu_joint: origin xyz=-0.032 0 0.068 rpy=0 0 0 -> xyz=-0.032 0 0.2136 rpy=0 0 0

Commit message: add anchors transform

File: pui_description/urdf/pui_bot.urdf (robot description, URDF)
Before this commit: robot pui_bot, 7 links, 6 joints
Links:
- added link anchor_0_link; visual box size=0.01 0.04 0.06
- added link anchor_1_link; visual box size=0.01 0.04 0.06
- added link anchor_2_link; visual box size=0.01 0.04 0.06
Joints:
- added joint anchor_0_joint: type fixed, parent base_link, child anchor_0_link, origin xyz=0.04 0 0.10 rpy=0 0 0
- added joint anchor_1_joint: type fixed, parent base_link, child anchor_1_link, origin xyz=0.8 0.30 0.35 rpy=0 0 0
- added joint anchor_2_joint: type fixed, parent base_link, child anchor_2_link, origin xyz=0.8 -0.30 0.35 rpy=0 0 0

Commit message: change anchor_0 default position

File: pui_description/urdf/pui_bot.urdf (robot description, URDF)
Before this commit: robot pui_bot, 10 links, 9 joints
Joints:
- joint anchor_0_joint: origin xyz=0.04 0 0.10 rpy=0 0 0 -> xyz=0.04 0.18 0.10 rpy=0 0 0

Commit message: change pui init position

File: pui_description/urdf/pui_bot.urdf (robot description, URDF)
Before this commit: robot pui_bot, 10 links, 9 joints
Joints:
- joint anchor_0_joint: origin xyz=0.04 0.18 0.10 rpy=0 0 0 -> xyz=-0.80 0.18 0.20 rpy=0 0 0

Commit message: debug anchor0 position

File: pui_description/urdf/pui_bot.urdf (robot description, URDF)
Before this commit: robot pui_bot, 10 links, 9 joints
Joints:
- joint anchor_0_joint: origin xyz=-0.80 0.18 0.20 rpy=0 0 0 -> xyz=-0.80 -0.18 0.20 rpy=0 0 0
