Commit message: tf for t2

File: pui_description/urdf/pui_t2.urdf (robot description, URDF)
Before this commit: robot pui_t2, 8 links, 7 joints
Links:
- removed link base_footprint
- removed link base_link
- removed link base_scan
- removed link caster_back_link
- removed link imu_link
- removed link tag_link
- removed link wheel_left_link
- removed link wheel_right_link
- added link t2/base_footprint
- added link t2/base_link, mass 8.2573504e-01; collision box size=0.140 0.140 0.143; visual mesh filename=package://pui_description/meshes/bases/burger_base.stl scale=0.001 0.001 0.001
- added link t2/caster_back_link, mass 0.005; collision box size=0.030 0.009 0.020
- added link t2/imu_link; visual mesh filename=package://pui_description/meshes/sensors/MTi_1.stl scale=0.001 0.001 0.001
- added link t2/tag_link; visual box size=0.01 0.04 0.06
- added link t2/wheel_left_link, mass 2.8498940e-02; collision cylinder length=0.018 radius=0.033; visual mesh filename=package://pui_description/meshes/wheels/left_tire.stl scale=0.001 0.001 0.001
- added link t2/wheel_right_link, mass 2.8498940e-02; collision cylinder length=0.018 radius=0.033; visual mesh filename=package://pui_description/meshes/wheels/right_tire.stl scale=0.001 0.001 0.001
Joints:
- removed joint base_joint
- removed joint caster_back_joint
- removed joint imu_joint
- removed joint scan_joint
- removed joint tag_joint
- removed joint wheel_left_joint
- removed joint wheel_right_joint
- added joint t2/base_joint: type fixed, parent t2/base_footprint, child t2/base_link, origin xyz=0.0 0.0 0.010 rpy=0 0 0
- added joint t2/caster_back_joint: type fixed, parent t2/base_link, child t2/caster_back_link, origin xyz=-0.081 0 -0.004 rpy=-1.57 0 0
- added joint t2/imu_joint: type fixed, parent t2/base_link, child t2/imu_link, origin xyz=-0.032 0 0.2136 rpy=0 0 0
- added joint t2/tag_joint: type fixed, parent t2/base_link, child t2/tag_link, origin xyz=0.0 -0.18 0.20 rpy=0 0 0
- added joint t2/wheel_left_joint: type continuous, parent t2/base_link, child t2/wheel_left_link, origin xyz=0.0 0.08 0.023 rpy=-1.57 0 0, axis 0 0 1
- added joint t2/wheel_right_joint: type continuous, parent t2/base_link, child t2/wheel_right_link, origin xyz=0.0 -0.080 0.023 rpy=-1.57 0 0, axis 0 0 1
